File: CAD/VFD_Controller/VFD_Controller.kicad_pcb (KiCad board)
At the start: 2 copper layers, 101.6 x 38.1 mm, 24 parts, among them IC1 PIC18F27Q10, J1 Barrel_Jack_Switch, J2 SB412A, J4 Conn_01x06, J5 ICSP, U1 AE-GPS, U2 M78AR033-1, U3 NJW4617

Commit message: v2 (working
Parts:
- C2: value 100u -> 22u; footprint Capacitor_SMD:CP_Elec_10x10 -> Capacitor_THT:CP_Radial_D6.3mm_P2.50mm
- IC1: footprint Package_DFN_QFN:QFN-28-1EP_6x6mm_P0.65mm_EP4.25x4.25mm_ThermalVias -> Package_DFN_QFN:QFN-28-1EP_6x6mm_P0.65mm_EP4.25x4.25mm
- moved C2 0.66 mm to (181.6, 106.0)
Connections:
- C5 pad 1: +24V -> +3V3
- U1 pad 3: Net-(U1-Pad3) -> +3V3
- U3 pad 1: +24V -> +3V3
Routing:
- net +24V: track 163.5 -> 145.5 mm, vias 1 -> 0
- net +3V3: track 154.9 -> 170.0 mm, vias 4 -> 5
- net GND: track 19.5 -> 5.90 mm, vias 95 -> 108
Other:
- board text added: "DC 24V/1A"
- board text removed: "DC 24V/2A"
