File: CAD/VFD_Driver/VFD_Driver.kicad_pcb (KiCad board)
At the start: 2 copper layers, 101.6 x 38.1 mm, 20 parts, among them IC1 MAX6922, IC2 MAX6922, J1 Conn_01x06, J2 Conn_01x06, Q1 IRLML6344

Commit message: v2 (working
Parts:
- removed D1, D2, D3: GS1010FL, Gentiana:SOD-123FL
- added IC3: TSR_2-0512, SamacSys_Parts:TSR22412, F.Cu at (133.6, 81.3)
- C1, C2, C3, C4: footprint Capacitor_SMD:C_0603_1608Metric_Pad1.08x0.95mm_HandSolder -> Capacitor_SMD:C_0603_1608Metric
- Q1: footprint Package_TO_SOT_SMD:SOT-23_Handsoldering -> Package_TO_SOT_SMD:SOT-23
- R1, R2: footprint Resistor_SMD:R_0603_1608Metric_Pad0.98x0.95mm_HandSolder -> Resistor_SMD:R_0603_1608Metric
- moved Q1 0.26 mm to (131.1, 93.0)
- moved R1 0.10 mm to (138.2, 94.0)
- moved C2 0.10 mm to (139.7, 83.3)
- moved C4 0.10 mm to (185.4, 83.3)
- moved R2 0.09 mm to (134.6, 93.2)
Routing:
- net +24V: track 174.5 -> 185.4 mm
- net /H_Power: track 114.7 -> 124.6 mm
- net GND: track 17.5 -> 25.0 mm, vias 128 -> 156
- net Net-(D2-Pad1): track 5.50 -> 0.00 mm
- net +3V3: track 92.0 -> 95.9 mm
- net Net-(D1-Pad1): track 3.38 -> 0.00 mm
- net /5_E: track 37.6 -> 38.5 mm
